Commit message: Implemented new map (medium 6 blocks)

File: BLG456EAssignment3/models/horizontal_block.urdf (robot description, URDF)
Before this commit: robot horizontal_block, 1 links, 0 joints
Links:
- removed link my_hor_block
- added link my_ver_block, mass 1.0; collision box size=1 5 2; visual box size=1 5 2

File: BLG456EAssignment3/models/vertical_block.urdf (robot description, URDF)
Before this commit: robot vertical_block, 1 links, 0 joints
Links:
- removed link my_ver_block
- added link my_hor_block, mass 1.0; collision box size=5 1 2; visual box size=5 1 2
